Commit message: fix bug of gap extractor

File: src/simple_robot/urdf/velodyne.xacro (robot description, xacro)
@@ -2,5 +2,5 @@
 <robot xmlns:xacro="http://www.ros.org/wiki/xacro" name="velodyne">
   <xacro:property name="M_PI" value="3.1415926535897931" />
-    <xacro:macro name="Velodyne-HDL-32E" params="connected_to scan_name xyz:='0 0 0' rpy:='0 0 0' topic:=/velodyne_points hz:=20 lasers:=16 samples:=1600 collision_range:=0.01 min_range:=0.01 max_range:=3.5 noise:=0.001 min_angle:=-${M_PI} max_angle:=${M_PI} gpu:=true">
+    <xacro:macro name="Velodyne-HDL-32E" params="connected_to scan_name xyz:='0 0 0' rpy:='0 0 0' topic:=/velodyne_points hz:=20 lasers:=32 samples:=1600 collision_range:=0.01 min_range:=0.01 max_range:=3.5 noise:=0.001 min_angle:=-${M_PI} max_angle:=${M_PI} gpu:=true">
         <xacro:arg name="velodyne-laser_visual"  default="false"/>
         <!-- scan is fixed to the base link -->
