Commit message: fix bug in freespace generation in 2D case(3D not test yet)

File: src/simple_robot/urdf/simple_robot.xacro (robot description, xacro)
@@ -8,5 +8,5 @@
     <visual>
       <geometry>
-        <box size="0.2 0.2 0.2"/>
+        <box size="0.4 0.2 0.2"/>
       </geometry>
       <material name="blue">

Commit message: update visulization

File: src/simple_robot/urdf/simple_robot.xacro (robot description, xacro)
@@ -23,4 +23,5 @@
     <gravity>false</gravity>
     <kinematic>true</kinematic>
+    <material>Gazebo/Blue</material>
   </gazebo>
   <xacro:if value="$(arg if_3D_Lidar)">
